Commit message: Added Task 2

File: ebot_description/models/ebot/ebot_description.xacro (robot description, xacro)
@@ -4,5 +4,5 @@
 *  Filename:           ebot.gazebo
 *  Description:        Gazebo Plugins
-*  Modified by:        Sahil
+*  Modified by:        Joel Devasia, Sahil
 *  Author:             e-Yantra Team
 *****************************************************************************************
@@ -46,8 +46,4 @@
     <inertial>
       <origin xyz="0 0.0 0.12" rpy="0 0 0" />
-      <!--       <mass
-        value="60" />
-         <inertia ixx="0.7625" ixy="0" ixz="0" iyy="2.0236" iyz="0" izz="2.1611"/>
- -->
       <xacro:box_inertia b_mass="${base_mass}" b_x="0.585" b_y="0.30" b_z="0.25" />
     </inertial>
@@ -57,6 +53,4 @@
         rpy="0 0 0" />
       <geometry>
-        <!-- <mesh
-          filename="file://$(find ebot_description)/meshes/chassis.dae" /> -->
           <mesh
           filename="file://$(find ebot_description)/meshes/chassis_modified.dae" />
@@ -69,4 +63,12 @@
       <geometry>
         <box size="0.585 0.30 0.25" />
+      </geometry>
+    </collision>
+    <collision>
+      <origin
+        xyz="0 0.0 0.457521"
+        rpy="0 0 0" />
+      <geometry>
+        <box size="0.35 0.29 0.435" />
       </geometry>
     </collision>
@@ -84,7 +86,4 @@
         xyz="6.6592E-05 0.025016 -1.3483E-06"
         rpy="0 0 0" />
-      <!--       <mass
-        value="2" />
-          <inertia ixx="0.0054" ixy="0" ixz="0" iyy="0.0054" iyz="0" izz="0.01"/> -->
       <xacro:insert_block name="wheel_inertia" />
     </inertial>
@@ -132,7 +131,4 @@
         xyz="6.6594E-05 0.025016 -1.349E-06"
         rpy="0 0 0" />
-      <!--      <mass
-        value="2" />
-          <inertia ixx="0.0054" ixy="0" ixz="0" iyy="0.0054" iyz="0" izz="0.01"/> -->
       <xacro:insert_block name="wheel_inertia" />
     </inertial>
@@ -180,7 +176,4 @@
         xyz="6.6592E-05 0.025016 -1.3483E-06"
         rpy="0 0 0" />
-      <!--       <mass
-        value="2" />
-          <inertia ixx="0.0054" ixy="0" ixz="0" iyy="0.0054" iyz="0" izz="0.01"/> -->
       <xacro:insert_block name="wheel_inertia" />
     </inertial>
@@ -228,7 +221,4 @@
         xyz="6.6594E-05 0.025016 -1.349E-06"
         rpy="0 0 0" />
-      <!--       <mass
-        value="2" />
-          <inertia ixx="0.0054" ixy="0" ixz="0" iyy="0.0054" iyz="0" izz="0.01"/> -->
       <xacro:insert_block name="wheel_inertia" />
     </inertial>
@@ -269,57 +259,7 @@
       xyz="0 1 0" />
   </joint>
-  <!-- Intel real sense Camera for 3D mapping-->
-  <!-- <joint name="realsensejoint" type="fixed">
-    <axis xyz="0 0 0" />
-    <origin xyz="0.277944460576403 0.00208437301780086 0.0230507258091751" rpy="0 0 0"/>
-    <parent link="ebot_base"/>
-    <child link="camera_link"/>
-  </joint>
-  <link name="camera_link">
-    <collision>
-      <origin xyz="0.02 0 0" rpy="0 0 0"/>
-      <geometry>0
-        <box size="0.001 0.001 0.001"/>
-      </geometry>
-    </collision>
-    <visual>
-      <origin xyz="0 0 0" rpy="1.5707 0 1.5707"/>
-      <geometry>
-        <mesh filename="file://$(find ebot_description)/meshes/NAVRS.STL" />
-      </geometry>
-    </visual>
-    <inertial>
-      <mass value="1e-5" />
-      <origin xyz="0 0 0" rpy="0 0 0"/>
-      <inertia ixx="0" ixy="0" ixz="0" iyy="0" iyz="0" izz="0" />
-    </inertial>
-  </link>
-  <joint name="camera_optical_joint" type="fixed">
-    <origin xyz="0 0 0" rpy="${-pi/2} 0 ${-pi/2}"/>
-    <parent link="camera_link"/>
-    <child link="camera_rgb_frame"/>
-  </joint>
-  <link name="camera_rgb_frame">
-  </link>
-  <joint name="camera_depth_joint" type="fixed">
-    <origin xyz="0 0 0" rpy="${-pi/2} 0 ${-pi/2}"/>
-    <parent link="camera_link"/>
-    <child link="camera_depth_frame"/>
-  </joint>
-    <link name="camera_depth_frame">
-  </link> -->
   <!-- LIDAR -->
   <link name="laser">
     <origin rpy="0 0 0" xyz="0 0 0" />
-    <!-- <inertial>
-      <mass value="0.09"/>
-      <inertia ixx="4.275e-05" ixy="0" ixz="0" iyy="4.275e-05" iyz="0" izz="5.5125e-05"/>
-    </inertial>
-    <collision>
-      <origin rpy="0 0 0" xyz="0 0 0"/>
-      <geometry>
-        <cylinder length="0.040" radius="0.030"/>
-      </geometry>
-    </collision> -->
     <visual>
       <origin rpy="0 0 0" xyz="0 0 0" />
@@ -342,18 +282,4 @@
   <link
     name="FUS1">
-    <!-- <inertial>
-      <origin
-        xyz="-0.00265918092876655 2.08166817117217E-17 0.0100193625139959"
-        rpy="0 0 0" />
-      <mass
-        value="0.0152532066391543" />
-      <inertia
-        ixx="4.77814992940302E-06"
-        ixy="-2.01819824421892E-21"
-        ixz="2.64657807499124E-08"
-        iyy="1.003384637723E-06"
-        iyz="-8.80528876343328E-21"
-        izz="4.55679776636487E-06" />
-    </inertial> -->
     <visual>
       <origin
@@ -370,12 +296,4 @@
       </material>
     </visual>
-    <!-- <collision>
-      <origin
-        xyz="0 0 0"
-        rpy="0 0 0" />
-      <geometry>
-          <box size="0.019 0.057 0.028"/>
-      </geometry>
-    </collision> -->
   </link>
   <joint
@@ -395,18 +313,4 @@
   <link
     name="FUS2">
-    <!-- <inertial>
-      <origin
-        xyz="-0.0026592 1.9949E-17 0.010019"
-        rpy="0 0 0" />
-      <mass
-        value="0.015253" />
-      <inertia
-        ixx="4.7781E-06"
-        ixy="-2.0925E-21"
-        ixz="2.6466E-08"
-        iyy="1.0034E-06"
-        iyz="-9.4695E-21"
-        izz="4.5568E-06" />
-    </inertial> -->
     <visual>
       <origin
@@ -423,12 +327,4 @@
       </material>
     </visual>
-    <!-- <collision>
-      <origin
-        xyz="0 0 0"
-        rpy="0 0 0" />
-      <geometry>
-           <box size="0.019 0.057 0.028"/>
-      </geometry>
-    </collision> -->
   </link>
   <joint
@@ -448,18 +344,4 @@
   <link
     name="FUS3">
-    <!-- <inertial>
-      <origin
-        xyz="-0.0026592 5.5511E-17 0.010019"
-        rpy="0 0 0" />
-      <mass
-        value="0.015253" />
-      <inertia
-        ixx="4.7781E-06"
-        ixy="2.7832E-20"
-        ixz="2.6466E-08"
-        iyy="1.0034E-06"
-        iyz="1.4502E-20"
-        izz="4.5568E-06" />
-    </inertial> -->
     <visual>
       <origin
@@ -476,12 +358,4 @@
       </material>
     </visual>
-    <!-- <collision>
-      <origin
-        xyz="0 0 0"
-        rpy="0 0 0" />
-      <geometry>
-           <box size="0.019 0.057 0.028"/>
-      </geometry>
-    </collision> -->
   </link>
   <joint
@@ -501,18 +375,4 @@
   <link
     name="FUS4">
-    <!-- <inertial>
-      <origin
-        xyz="-0.00265918092876644 6.93889390390723E-17 0.0100193625139959"
-        rpy="0 0 0" />
-      <mass
-        value="0.0152532066391543" />
-      <inertia
-        ixx="4.77814992940302E-06"
-        ixy="2.8163959262392E-20"
-        ixz="2.64657807499109E-08"
-        iyy="1.003384637723E-06"
-        iyz="2.09456577324828E-20"
-        izz="4.55679776636487E-06" />
-    </inertial> -->
     <visual>
       <origin
@@ -529,12 +389,4 @@
       </material>
     </visual>
-    <!-- <collision>
-      <origin
-        xyz="0 0 0"
-        rpy="0 0 0" />
-      <geometry>
-           <box size="0.019 0.057 0.028"/>
-      </geometry>
-    </collision> -->
   </link>
   <joint
@@ -558,18 +410,4 @@
   <link
     name="ultrasonic_rl">
-    <!-- <inertial>
-      <origin
-        xyz="-0.0026592 2.6021E-17 0.010019"
-        rpy="0 0 0" />
-      <mass
-        value="0.015253" />
-      <inertia
-        ixx="4.7781E-06"
-        ixy="-1.9723E-21"
-        ixz="2.6466E-08"
-        iyy="1.0034E-06"
-        iyz="-7.7105E-21"
-        izz="4.5568E-06" />
-    </inertial> -->
     <visual>
       <origin
@@ -586,12 +424,4 @@
       </material>
     </visual>
-    <!-- <collision>
-      <origin
-        xyz="0 0 0"
-        rpy="0 0 0" />
-      <geometry>
-           <box size="0.019 0.057 0.028"/>
-      </geometry>
-    </collision> -->
   </link>
   <joint
@@ -614,18 +444,4 @@
   <link
     name="ultrasonic_rr">
-    <!-- <inertial>
-      <origin
-        xyz="-0.00265918092876644 2.34187669256869E-17 0.0100193625139959"
-        rpy="0 0 0" />
-      <mass
-        value="0.0152532066391543" />
-      <inertia
-        ixx="4.77814992940302E-06"
-        ixy="-1.34867897211379E-21"
-        ixz="2.64657807499114E-08"
-        iyy="1.003384637723E-06"
-        iyz="-1.29818552470248E-20"
-        izz="4.55679776636487E-06" />
-    </inertial> -->
     <visual>
       <origin
@@ -642,12 +458,4 @@
       </material>
     </visual>
-    <!-- <collision>
-      <origin
-        xyz="0 0 0"
-        rpy="0 0 0" />
-      <geometry>
-           <box size="0.019 0.057 0.028"/>
-      </geometry>
-    </collision> -->
   </link>
   <joint
@@ -667,18 +475,4 @@
   <link
     name="RHUS7">
-    <!-- <inertial>
-      <origin
-        xyz="-0.00265918092876641 1.23570598198341E-12 0.0100193625139959"
-        rpy="0 0 0" />
-      <mass
-        value="0.0152532066391543" />
-      <inertia
-        ixx="4.77814992940302E-06"
-        ixy="3.27217392921119E-18"
-        ixz="2.64657807499107E-08"
-        iyy="1.003384637723E-06"
-        iyz="4.38229124201629E-16"
-        izz="4.55679776636487E-06" />
-    </inertial> -->
     <visual>
       <origin
@@ -695,12 +489,4 @@
       </material>
     </visual>
-    <!-- <collision>
-      <origin
-        xyz="0 0 0"
-        rpy="0 0 0" />
-      <geometry>
-           <box size="0.019 0.057 0.028"/>
-      </geometry>
-    </collision> -->
   </link>
   <joint
@@ -720,18 +506,4 @@
   <link
     name="RHUS9">
-    <!-- <inertial>
-      <origin
-        xyz="-0.0026592 6.9389E-18 0.010019"
-        rpy="0 0 0" />
-      <mass
-        value="0.015253" />
-      <inertia
-        ixx="4.7781E-06"
-        ixy="1.6008E-20"
-        ixz="2.6466E-08"
-        iyy="1.0034E-06"
-        iyz="-1.185E-20"
-        izz="4.5568E-06" />
-    </inertial> -->
     <visual>
       <origin
@@ -748,12 +520,4 @@
       </material>
     </visual>
-    <!-- <collision>
-      <origin
-        xyz="0 0 0"
-        rpy="0 0 0" />
-      <geometry>
-           <box size="0.019 0.057 0.028"/>
-      </geometry>
-    </collision> -->
   </link>
   <joint
@@ -773,18 +537,4 @@
   <link
     name="LHUS9">
-    <!-- <inertial>
-      <origin
-        xyz="-0.00265918092876642 -1.2353174039248E-12 0.0100193625139958"
-        rpy="0 0 0" />
-      <mass
-        value="0.0152532066391543" />
-      <inertia
-        ixx="4.77814992940302E-06"
-        ixy="-3.2538981368926E-18"
-        ixz="2.64657807499116E-08"
-        iyy="1.003384637723E-06"
-        iyz="-4.38135627183199E-16"
-        izz="4.55679776636487E-06" />
-    </inertial> -->
     <visual>
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
File: ur_description/urdf/ur.urdf.xacro (robot description, xacro)
@@ -124,4 +124,14 @@
     <origin xyz="-1.08 0.007 1.09" rpy="0.0 0.7330383 0.0" />
 </xacro:realsense2_camera>
+ <gazebo reference="wrist_3_link">
+     <sensor name="ft_sensor" type="force_torque">
+       <always_on>true</always_on>
+       <update_rate>500</update_rate>
+       <topic>/ur5/ft_sensor</topic>
+       <force_torque>
+         <frame>child</frame>
+       </force_torque>
+     </sensor>
+   </gazebo>
 <!-- Remove your manual camera_link definition -->
   <!-- <xacro:include filename="$(find ur_description)/urdf/realsense2.urdf.xacro" />

File: ur_description/urdf/ur_macro.xacro (robot description, xacro)
@@ -399,18 +399,23 @@
       <inertia ixx="1e-6" ixy="0.0" ixz="0.0" iyy="1e-6" iyz="0.0" izz="1e-6"/>
     </inertial>
+    <sensor name="wrist_ft" type="force_torque">
+    <update_rate>500</update_rate>
+    <topic>/ur5/wrist_ft</topic>
+    <force_torque>
+      <frame>child</frame>
+    </force_torque>
+  </sensor>
     </link>
     <gazebo reference="${tf_prefix}wrist_3_joint">
         <sensor name="force_torque_sensor" type="force_torque">
-          <always_on>true</always_on>
-          <update_rate>100</update_rate>
-          <visualize>true</visualize>
-          <topic>force_torque</topic>
-          <enable_metrics>true</enable_metrics>
-          <pose>0 0 0 0 0 0</pose>
-          <force_torque>
-            <frame>sensor</frame>
-            <measure_direction>child_to_parent</measure_direction>
-          </force_torque>
-        </sensor>
+        <always_on>true</always_on>
+        <update_rate>50</update_rate>
+        <visualize>true</visualize>
+        <topic>force_torque/eef</topic>
+        <force_torque>
+          <frame>sensor</frame>
+          <measure_direction>parent_to_child</measure_direction>
+        </force_torque>
+      </sensor>
     </gazebo>
   </xacro:macro>
